Commit message: Add files via upload

File: gazebo_demo/urdf/ABot.urdf.xacro (robot description, xacro)
@@ -1,11 +1,54 @@
-<?xml version="1.0"?>
-<robot xmlns:xacro="http://www.ros.org/wiki/xacro" name="ABot">
-  <!--<link name="base_footprint">
-   </link>
-  <joint name="base_footprint_joint" type="fixed">
-     <parent link="base_footprint"/>
-     <child link="base_link"/>
-     <origin xyz="0.00 0.00 0.1" rpy="0.0 0.0 0.0"/>
-   </joint>-->
+<?xml version='1.0'?>
+<robot name="ABot" xmlns:xacro="http://www.ros.org/wiki/xacro">
+<xacro:include filename="$(find gazebo_demo)/urdf/ABot_kinect.xacro"/>
+<!-- RGBD Camera -->
+  <gazebo reference="kinect_baselink"> <!-- reference must match the name of the link in the Xacro URDF -->
+    <sensor type="depth" name="camera1"> <!-- The name must be unique from all other sensor names -->
+        <always_on>1</always_on>
+        <update_rate>20.0</update_rate>
+        <visualize>true</visualize>
+        <camera>
+            <horizontal_fov>1.047</horizontal_fov>
+            <image>
+                <width>640</width>
+                <height>480</height>
+                <format>R8G8B8</format>
+            </image>
+            <depth_camera>
+            </depth_camera>
+            <clip>
+                <near>0.1</near>
+                <far>20</far>
+            </clip>
+        </camera>
+             <!-- link to the camera's shared object file -->
+             <plugin name="camera_controller" filename="libgazebo_ros_openni_kinect.so">
+             <alwaysOn>true</alwaysOn>
+                <updateRate>10.0</updateRate>
+                <!-- namespaces to avoid collision with other topics -->
+                <cameraName>camera</cameraName>
+                <!-- The coordinate frame the point cloud image is published under in the tf tree -->
+                <!-- Rotate this frame in urdf/xacro file if point cloud is not correctly oriented in Rviz -->
+                <frameName>camera_rgbd_frame</frameName>
+            <!--topic the camera will be publishing to (image, info, depth image, point cloud -->
+            <imageTopicName>rgb/image_raw</imageTopicName>
+            <depthImageTopicName>depth/image_raw</depthImageTopicName>
+            <pointCloudTopicName>depth/points</pointCloudTopicName>
+            <cameraInfoTopicName>rgb/camera_info</cameraInfoTopicName>
+            <depthImageCameraInfoTopicName>depth/camera_info</depthImageCameraInfoTopicName>
+            <pointCloudCutoff>0.4</pointCloudCutoff>
+                <hackBaseline>0.07</hackBaseline>
+                <distortionK1>0.0</distortionK1>
+                <distortionK2>0.0</distortionK2>
+                <distortionK3>0.0</distortionK3>
+                <distortionT1>0.0</distortionT1>
+                <distortionT2>0.0</distortionT2>
+            <CxPrime>0.0</CxPrime>
+            <Cx>0.0</Cx>
+            <Cy>0.0</Cy>
+            <focalLength>0.0</focalLength>
+            </plugin>
+    </sensor>
+  </gazebo>
   <link name="base_link">
   <inertial>
@@ -27,34 +70,4 @@
   </collision>
   </link>
-<!--
-   <link name="box">
-  <inertial>
-    <origin xyz="0 0 0" />
-    <mass value="5" />
-    <inertia  ixx="0.1" ixy="0.0"  ixz="0.0"  iyy="0.1"  iyz="0.0"  izz="0.1" />
-  </inertial>
-  <visual>
-    <origin xyz="0 0 0"/>
-    <geometry>
-      <box size="0.3 0.2 0.1" />
-    </geometry>
-  </visual>
-  <collision>
-    <origin xyz="0 0 0"/>
-    <geometry>
-      <box size="0.3 0.2 0.1" />
-    </geometry>
-  </collision>
-  </link>
-  <gazebo reference="box">
-    <material>Gazebo/Black</material>
-  </gazebo>
-  <joint name="base_link_box" type="fixed">
-    <parent link="base_link"/>
-    <child link="box"/>
-    <axis xyz="0 0 0"/>
-    <origin xyz="-0.05 0 0.225"/>
-  </joint>
--->
   <gazebo reference="base_link">
     <material>Gazebo/DarkGrey</material>
@@ -219,30 +232,10 @@
     </inertial>
   </link>
-<joint name="hokuyo_joint" type="fixed">
+<joint name="kinect_joint" type="fixed">
     <axis xyz="0 1 0" />
     <origin xyz="0.15 0 0.2" rpy="0 0 0"/>
     <parent link="base_link"/>
-    <child link="hokuyo_link"/>
-  </joint>
-  <!-- Hokuyo Laser -->
-  <link name="hokuyo_link">
-    <collision>
-      <origin xyz="0 0 0" rpy="0 0 0"/>
-      <geometry>
-    <box size="0.1 0.1 0.1"/>
-      </geometry>
-    </collision>
-    <visual>
-      <origin xyz="0 0 0" rpy="0 0 0"/>
-      <geometry>
-        <mesh filename="package://gazebo_demo/urdf/hokuyo.dae"/>
-      </geometry>
-    </visual>
-    <inertial>
-      <mass value="1e-5" />
-      <origin xyz="0 0 0" rpy="0 0 0"/>
-      <inertia ixx="1e-6" ixy="0" ixz="0" iyy="1e-6" iyz="0" izz="1e-6" />
-    </inertial>
-  </link>
+    <child link="kinect_baselink"/>
+  </joint>
 <joint name="camera_joint" type="fixed">
     <axis xyz="0 0 0" />
@@ -352,39 +345,4 @@
   </plugin>
 </gazebo>
- <gazebo reference="hokuyo_link">
-    <sensor type="gpu_ray" name="head_hokuyo_sensor">
-      <pose>0 0 0 0 0 0</pose>
-      <visualize>false</visualize>
-      <update_rate>10</update_rate>
-      <ray>
-        <scan>
-          <horizontal>
-            <samples>720</samples>
-            <resolution>1</resolution>
-            <min_angle>-1.570796</min_angle>
-            <max_angle>1.570796</max_angle>
-          </horizontal>
-        </scan>
-        <range>
-          <min>0.10</min>
-          <max>20.0</max>
-          <resolution>0.01</resolution>
-        </range>
-        <noise>
-          <type>gaussian</type>
-          <!-- Noise parameters based on published spec for Hokuyo laser
-               achieving "+-30mm" accuracy at range < 10m.  A mean of 0.0m and
-               stddev of 0.01m will put 99.7% of samples within 0.03m of the true
-               reading. -->
-          <mean>0.0</mean>
-          <stddev>0.01</stddev>
-        </noise>
-      </ray>
-      <plugin name="gazebo_ros_head_hokuyo_controller" filename="libgazebo_ros_gpu_laser.so">
-        <topicName>scan</topicName>
-        <frameName>hokuyo_link</frameName>
-      </plugin>
-    </sensor>
-  </gazebo>
   <xacro:property name="hokuyo_link" value="0.05" />
   <xacro:property name="camera_link" value="0.05" />

Commit message: Add files via upload

File: gazebo_demo/urdf/ABot.urdf.xacro (robot description, xacro)
@@ -4,7 +4,7 @@
 <!-- RGBD Camera -->
   <gazebo reference="kinect_baselink"> <!-- reference must match the name of the link in the Xacro URDF -->
-    <sensor type="depth" name="camera1"> <!-- The name must be unique from all other sensor names -->
+    <sensor type="depth" name="kinect"> <!-- The name must be unique from all other sensor names -->
         <always_on>1</always_on>
-        <update_rate>20.0</update_rate>
+        <update_rate>30.0</update_rate>
         <visualize>true</visualize>
         <camera>
@@ -18,23 +18,23 @@
             </depth_camera>
             <clip>
-                <near>0.1</near>
+                <near>0.05</near>
                 <far>20</far>
             </clip>
         </camera>
              <!-- link to the camera's shared object file -->
-             <plugin name="camera_controller" filename="libgazebo_ros_openni_kinect.so">
+             <plugin name="kinect_controller" filename="libgazebo_ros_openni_kinect.so">
              <alwaysOn>true</alwaysOn>
-                <updateRate>10.0</updateRate>
+                <updateRate>30.0</updateRate>
                 <!-- namespaces to avoid collision with other topics -->
-                <cameraName>camera</cameraName>
+                <cameraName>kinect</cameraName>
                 <!-- The coordinate frame the point cloud image is published under in the tf tree -->
                 <!-- Rotate this frame in urdf/xacro file if point cloud is not correctly oriented in Rviz -->
-                <frameName>camera_rgbd_frame</frameName>
+                <frameName>camera_link</frameName>
             <!--topic the camera will be publishing to (image, info, depth image, point cloud -->
-            <imageTopicName>rgb/image_raw</imageTopicName>
-            <depthImageTopicName>depth/image_raw</depthImageTopicName>
-            <pointCloudTopicName>depth/points</pointCloudTopicName>
-            <cameraInfoTopicName>rgb/camera_info</cameraInfoTopicName>
-            <depthImageCameraInfoTopicName>depth/camera_info</depthImageCameraInfoTopicName>
+            <imageTopicName>/camera/image_raw</imageTopicName>
+            <depthImageTopicName>/kinect/depth/image_raw</depthImageTopicName>
+            <pointCloudTopicName>/kinect/depth/points</pointCloudTopicName>
+            <cameraInfoTopicName>/kinect/color/camera_info</cameraInfoTopicName>
+            <depthImageCameraInfoTopicName>/kinect/depth/camera_info</depthImageCameraInfoTopicName>
             <pointCloudCutoff>0.4</pointCloudCutoff>
                 <hackBaseline>0.07</hackBaseline>
@@ -345,5 +345,5 @@
   </plugin>
 </gazebo>
-  <xacro:property name="hokuyo_link" value="0.05" />
+  <xacro:property name="kinect_baselink" value="0.05" />
   <xacro:property name="camera_link" value="0.05" />
   <xacro:property name="camera_link_2" value="0.05" />

File: gazebo_demo/urdf/ABot_kinect.xacro (robot description, xacro)
@@ -41,5 +41,5 @@
        <origin xyz="0 0 0" rpy="-1.57079 0 3.14159"/>
         <geometry>
-         <mesh filename="package://rtab_dumpster/meshes/kinect.dae" scale="1.0 1.0 1.0"/>
+         <mesh filename="package://gazebo_demo/urdf/kinect.dae" scale="1.0 1.0 1.0"/>
         </geometry>
       </visual>
